File: kicad/OrangePiZeroExtentionBoard.sch (KiCad schematic (older format))
At the start: 54 parts, among them J10 PWM_OUT1, J11 CONN_UART, J12 PWM_OUT2, J13 FAN_12/24v, J15 PWM_OUT3, J2 DC_INPUT, J3 CONN_ADXL345, J4 OrangePi Zero GPIO PINs, J5 Conn_MAX31865, J7 OrangePi Zero Function Interf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

Commit message: update pin head footprint
Parts:
- J4: LCSC Part# C64320 -> (none)
- J7: LCSC Part# C52709 -> (none)
- USB1: symbol JerryKiCAD:USB_A_Port_x2 -> OrangePiZeroExtentionBoard-rescue:USB_A_Port_x2-JerryKiCAD
Changed lines of the file:
@@
 F 6 "J4" H 2050 3600 50  0001 C CNN "Reference"
 F 7 "OrangePi Zero GPIO PINs" H 2050 3600 50  0001 C CNN "Value"
-F 8 "C64320" H 2050 3600 50  0001 C CNN "LCSC Part#"
+F 8 "" H 2050 3600 50  0001 C CNN "LCSC Part#"
 	1    2050 3600
 	1    0    0    -1
@@
 F 6 "J7" H 4300 3600 50  0001 C CNN "Reference"
 F 7 "OrangePi Zero Function Interface" H 4300 3600 50  0001 C CNN "Value"
-F 8 "C52709" H 4300 3600 50  0001 C CNN "LCSC Part#"
+F 8 "" H 4300 3600 50  0001 C CNN "LCSC Part#"
 	1    4300 3600
 	1    0    0    -1
@@
 	2050 1150 2950 1150
 $Comp
-L JerryKiCAD:USB_A_Port_x2 USB1
+L OrangePiZeroExtentionBoard-rescue:USB_A_Port_x2-JerryKiCAD USB1
 U 1 1 61F6FF4E
 P 2600 6950
