File: kicad/OrangePiZeroExtentionBoard.kicad_pcb (KiCad board)
At the start: 4 copper layers, 85 x 56 mm, 54 parts, among them J10 PWM_OUT1, J11 CONN_UART, J12 PWM_OUT2, J13 FAN_12/24v, J15 PWM_OUT3, J2 DC_INPUT, J3 CONN_ADXL345, J4 OrangePi Zero GPIO PINs, J5 Conn_MAX31865, J7 OrangePi Zero Function Interf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

Commit message: updated
Routing:
- net GND: track 98.8 -> 79.9 mm, vias 27 -> 28
- net GPIO_0_SDI: track 64.6 -> 68.7 mm
- net GPIO_1_CS: track 68.7 -> 72.4 mm
- net GPIO_3_SDO: track 66.3 -> 69.2 mm
- net USB_DM3: track 28.7 -> 31.5 mm
- net USB_DP3: track 32.0 -> 34.1 mm
- net BUCK_BOOT: track 4.94 -> 5.82 mm
- net BUCK_PH: track 21.9 -> 22.5 mm
- net BUCK_IN: track 33.5 -> 34.0 mm
- net SPI1_MOSI: track 10.4 -> 10.9 mm, vias 0 -> 2
- net SPI1_MISO: track 9.42 -> 9.74 mm, vias 2 -> 0
- net SPI1_CS: track 16.4 -> 16.2 mm, vias 2 -> 0
Other:
- board text added: "POWER"
- board text removed: "PWR_LED"

Commit message: update details
Parts:
- moved R11 6.05 mm to (181.6, 95.9), turned to 270 degrees
- moved C1 4.32 mm to (170.5, 76.0)
- moved C3 1.12 mm to (173.0, 76.0)
Routing:
- net USB_DM3: track 31.5 -> 25.9 mm
- net BUCK_VSNS: track 21.5 -> 17.2 mm
- net +5V: track 56.7 -> 59.9 mm
- net GND: track 79.9 -> 81.7 mm
- net Net-(D5-Pad1): track 18.1 -> 19.2 mm
- net SPI1_CS: track 16.2 -> 16.8 mm
