File: kicad/orange_juice_board.kicad_pcb (KiCad board)
At the start: 4 copper layers, 85 x 56 mm, 54 parts, among them J10 PWM_OUT1, J11 CONN_UART, J12 PWM_OUT2, J13 FAN_12/24v, J15 PWM_OUT3, J2 DC_INPUT, J3 CONN_ADXL345, J4 OrangePi Zero GPIO PINs, J5 Conn_MAX31865, J7 OrangePi Zero Function Interf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

Commit message: update gerber
Routing:
- added copper zone on B.Cu, net GND
- added copper zone on F.Cu, net GND
Other:
- board text added: "Orange Juice v0.2 Design By Jerry"
- board text removed: "Orange Juice v0.1 Design by Jerry"

Commit message: version 0.3
Parts:
- moved C5 14.7 mm to (170.2, 91.9), turned to -90 degrees
- moved R11 13.3 mm to (168.9, 100.0), turned to 0 degrees
- moved D4 13.1 mm to (181.6, 96.6), turned to 0 degrees
- moved R13 12.1 mm to (168.9, 106.7), turned to 0 degrees
- moved R12 11.8 mm to (168.9, 102.9), turned to 180 degrees
- moved C4 10.5 mm to (174.9, 97.8), turned to 0 degrees
- moved Q1 8.90 mm to (181.0, 108.9)
- moved L1 8.75 mm to (178.6, 89.5), turned to 180 degrees
- moved C2 8.26 mm to (182.1, 102.9)
- moved R3 7.70 mm to (173.1, 108.0), turned to 180 degrees
- moved C3 5.42 mm to (170.5, 80.8), turned to 180 degrees
- moved R2 4.38 mm to (176.9, 108.0), turned to 180 degrees
- moved U1 3.94 mm to (175.3, 102.9), turned to 0 degrees
- moved C1 2.23 mm to (170.5, 78.2), turned to 180 degrees
- moved R1 1.23 mm to (182.9, 113.4), turned to -90 degrees
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- renumbered H2 to ?, H3 to ?, H4 to ?, H1 to ?
Connections:
- J4 pad 1: (no net) -> unconnected-(J4-Pad1)
- J4 pad 12: (no net) -> unconnected-(J4-Pad12)
- J4 pad 3: (no net) -> unconnected-(J4-Pad3)
- J4 pad 5: (no net) -> unconnected-(J4-Pad5)
- J4 pad 7: (no net) -> unconnected-(J4-Pad7)
- J7 pad 1: (no net) -> unconnected-(J7-Pad1)
- J7 pad 2: (no net) -> unconnected-(J7-Pad2)
- J7 pad 3: (no net) -> unconnected-(J7-Pad3)
- J7 pad 4: (no net) -> unconnected-(J7-Pad4)
- J7 pad 5: (no net) -> unconnected-(J7-Pad5)
- J7 pad 6: (no net) -> unconnected-(J7-Pad6)
- J7 pad 7: (no net) -> unconnected-(J7-Pad7)
- U1 pad 2: (no net) -> unconnected-(U1-Pad2)
- U1 pad 3: (no net) -> unconnected-(U1-Pad3)
- USB1 pad 9: Net-(USB1-Pad9) -> unconnected-(USB1-Pad9)
Routing:
- net GND: track 81.7 -> 0.14 mm, vias 28 -> 0
- net +5V: track 59.9 -> 13.0 mm, vias 4 -> 9
- net BUCK_IN: track 34.0 -> 8.97 mm, vias 0 -> 2
- net BUCK_PH: track 22.5 -> 0.00 mm
- net BUCK_VSNS: track 17.2 -> 7.33 mm, vias 2 -> 0
- net DCIN: track 10.6 -> 3.95 mm, vias 6 -> 3
- net USB_DP3: track 33.7 -> 29.2 mm
- net USB_DP2: track 22.6 -> 20.6 mm, vias 2 -> 0
- net USB_DM2: track 19.2 -> 20.9 mm, vias 0 -> 1
- net BUCK_EN: track 8.15 -> 6.60 mm
- net Net-(D5-Pad1): track 19.2 -> 17.8 mm
- net BUCK_BOOT: track 5.82 -> 4.36 mm
- net +3V3: track 76.4 -> 75.1 mm
- net Net-(Q4-Pad1): track 67.9 -> 68.6 mm
- net UART1_TX: track 12.5 -> 11.8 mm
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- added copper zone on F.Cu, net +5V
- added copper zone on F.Cu, net BUCK_IN
- added copper zone on F.Cu, net BUCK_PH
- added copper zone on F.Cu, net DCIN
Other:
- net class Default removed
- board text added: "For Orangepi zero with klipper features"
- board text added: "Orange Juice v0.3 Design By Jerry"
- board text removed: "Orange Juice v0.2 Design By Jerry"
