File: kicad/orange_juice_board.kicad_pcb (KiCad board)
At the start: 2 copper layers, 85 x 56 mm, 62 parts, among them J10 PWM_OUT1, J11 CONN_UART, J12 PWM_OUT2, J13 FAN_12/24v, J15 PWM_OUT3, J2 DC_INPUT, J3 CONN_ADXL345, J4 OrangePi Zero GPIO PINs, J5 Conn_MAX31865, J7 OrangePi Zero Function Interf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

Commit message: update v0.6
Parts:
- added D6: D_TVS, Diode_SMD:D_SMB, F.Cu at (154.4, 105.8)
- added Q5: MMBT5401, Package_TO_SOT_SMD:SOT-23, F.Cu at (154.2, 79.2)
- added Q6: SI2305A, Package_TO_SOT_SMD:SOT-23, F.Cu at (148.5, 75.5)
- added Q7: SI2305A, Package_TO_SOT_SMD:SOT-23, F.Cu at (150.4, 79.4)
- added R8: 100, Resistor_SMD:R_0805_2012Metric, F.Cu at (152.2, 74.3)
- added R8: 100, Resistor_SMD:R_0805_2012Metric, F.Cu at (152.2, 76.4)
- J12: renamed from J5; value Conn_MAX31865 -> Conn_01x08; footprint Connector_PinSocket_2.54mm:PinSocket_1x06_P2.54mm_Vertical -> Connector_PinSocket_2.54mm:PinSocket_1x08_P2.54mm_Vertical
- moved C4 13.1 mm to (152.6, 83.5), turned to -90 degrees
- moved C5 11.1 mm to (154.7, 83.5), turned to -90 degrees
- moved J12 2.53 mm to (148.9, 83.7)
- moved D1 1.92 mm to (156.7, 100.7)
- moved R5 1.84 mm to (153.4, 101.1), turned to 180 degrees
- moved C1 0.98 mm to (156.9, 72.1)
- moved C3 0.90 mm to (156.9, 74.2)
Connections:
- C1 pad 1: BUCK_OUT -> HATDC_5V
- C3 pad 1: BUCK_OUT -> HATDC_5V
- J12 pad 1: GND -> unconnected-(J12-Pad1)
- J12 pad 2: +3V3 -> GND
- J12 pad 3: GPIO_2_CLK -> PI_3.3V
- J12 pad 4: GPIO_3_SDO -> GPIO_2_CLK
- J12 pad 5: GPIO_0_SDI -> GPIO_3_SDO
- J12 pad 6: GPIO_1_CS -> GPIO_0_SDI
- J3 pad 2: +3V3 -> PI_3.3V
- J4 pad 17: +3V3 -> PI_3.3V
- J4 pad 2: BUCK_OUT -> HATDC_5V
- J4 pad 4: BUCK_OUT -> HATDC_5V
- J8 pad 1: BUCK_OUT -> HATDC_5V
- J9 pad 1: BUCK_OUT -> HATDC_5V
- USB1 pad 1: BUCK_OUT -> HATDC_5V
- USB1 pad 5: BUCK_OUT -> HATDC_5V
- USB1 pad 9: GND -> unconnected-(USB1-Pad9)
Routing:
- net HATDC_5V: track 0.00 -> 141.4 mm, vias 0 -> 8
- net BUCK_OUT: track 145.1 -> 22.2 mm, vias 9 -> 0
- net PI_3.3V: track 0.00 -> 79.8 mm, vias 0 -> 1
- net +3V3: track 79.8 -> 0.00 mm, vias 1 -> 0
- net BUCK_IN: track 125.3 -> 134.0 mm, vias 11 -> 10
- net Net-(Q6-Pad1): track 0.00 -> 7.51 mm
- net USB_DM3: track 28.0 -> 32.8 mm
- net Net-(Q5-Pad1): track 0.00 -> 4.16 mm
- net USB_DP3: track 29.7 -> 32.7 mm, vias 1 -> 0
- net Net-(D1-Pad2): track 5.24 -> 8.00 mm
- net USB_DP2: track 21.5 -> 19.9 mm, vias 1 -> 0
- net BUCK_BST: track 3.93 -> 4.55 mm
- net USB_DM2: track 20.2 -> 19.8 mm, vias 0 -> 1
- net GND: vias 4 -> 5
- added copper zone on F.Cu, net HATDC_5V
Other:
- board text added: "Orange Juice v0.5 Design by Jerry for klipper B站：大石头Jerry"

Commit message: update to v0.6
Parts:
- D6: value D_TVS -> SMAJ24A
- turned D6 to 180 degrees
Connections:
- D6 pad 1: GND -> DC_IN
- D6 pad 2: DC_IN -> GND
Routing:
- net GND: vias 5 -> 7
Changed lines of the file:
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@@
   )
   (footprint "Diode_SMD:D_SMB" (layer "F.Cu")
-    (at 154.4 105.8)
+    (at 154.4 105.8 180)
     (descr "Diode SMB (DO-214AA)")
     (tags "Diode SMB (DO-214AA)")
@@
       (effects (font (size 1 1) (thickness 0.15)))
     )
-    (fp_text value "D_TVS" (at 0 3.1) (layer "F.Fab")
+    (fp_text value "SMAJ24A" (at 0 3.1) (layer "F.Fab")
       (effects (font (size 1 1) (thickness 0.15)))
     )
@@
     (fp_line (start 0.50118 0.75032) (end 0.50118 -0.79908) (layer "F.Fab") (width 0.1))
     (fp_line (start 2.3 2) (end -2.3 2) (layer "F.Fab") (width 0.1))
-    (pad "1" smd rect locked (at -2.15 0) (size 2.5 2.3) (layers "F.Cu" "F.Paste" "F.Mask")
-      (net 2 "GND") (pinfunction "A1") (pintype "passive"))
-    (pad "2" smd rect locked (at 2.15 0) (size 2.5 2.3) (layers "F.Cu" "F.Paste" "F.Mask")
-      (net 15 "DC_IN") (pinfunction "A2") (pintype "passive"))
+    (pad "1" smd rect locked (at -2.15 0 180) (size 2.5 2.3) (layers "F.Cu" "F.Paste" "F.Mask")
+      (net 15 "DC_IN") (pinfunction "A1") (pintype "passive"))
+    (pad "2" smd rect locked (at 2.15 0 180) (size 2.5 2.3) (layers "F.Cu" "F.Paste" "F.Mask")
+      (net 2 "GND") (pinfunction "A2") (pintype "passive"))
     (model "${KICAD6_3DMODEL_DIR}/Diode_SMD.3dshapes/D_SMB.wrl"
       (offset (xyz 0 0 0))
@@
   )
   (footprint "Resistor_SMD:R_0805_2012Metric" (layer "F.Cu")
-    (at 153.3875 101.1 180)
+    (at 153.4 101.1 180)
     (descr "Resistor SMD 0805 (2012 Metric), square (rectangular) end terminal, IPC_7351 nominal, (Body size source: IPC-SM-782 page 72, https://www.pcb-3d.com/wordpress/wp-content/uploads/ipc-sm-782a_amendment_1_and_2.pdf), generated with kicad-footprint-generator")
     (tags "resistor")
@@
   (segment (start 98.7 104.0625) (end 98.6625 104.1) (width 0.25) (layer "F.Cu") (net 2))
   (via (at 106.934 104.521) (size 0.8) (drill 0.4) (layers "F.Cu" "B.Cu") (free) (net 2))
+  (via (at 157.85 98.1) (size 0.8) (drill 0.4) (layers "F.Cu" "B.Cu") (free) (net 2))
   (via (at 106.934 103.759) (size 0.8) (drill 0.4) (layers "F.Cu" "B.Cu") (free) (net 2))
+  (via (at 159.65 98.1) (size 0.8) (drill 0.4) (layers "F.Cu" "B.Cu") (free) (net 2))
   (via (at 105.537 104.521) (size 0.8) (drill 0.4) (layers "F.Cu" "B.Cu") (free) (net 2))
   (via (at 152.35 75.35) (size 0.8) (drill 0.4) (layers "F.Cu" "B.Cu") (free) (net 2))
@@
   (segment (start 156.051642 97.023) (end 156.0595 97.015142) (width 0.25) (layer "F.Cu") (net 7))
   (segment (start 154.3285 97.0605) (end 154.366 97.023) (width 0.25) (layer "F.Cu") (net 7))
-  (segment (start 154.666 100.966) (end 154.432 101.2) (width 0.25) (layer "F.Cu") (net 8))
-  (segment (start 154.3 101.1) (end 154.65 100.75) (width 0.25) (layer "F.Cu") (net 8))
+  (segment (start 154.3125 101.1) (end 156.25 101.1) (width 0.25) (layer "F.Cu") (net 8))
   (segment (start 158.95 99.05) (end 159.15 99.25) (width 0.25) (layer "F.Cu") (net 8))
   (segment (start 156.7 99.05) (end 158.95 99.05) (width 0.25) (layer "F.Cu") (net 8))
+  (segment (start 156.25 101.1) (end 156.7 100.65) (width 0.25) (layer "F.Cu") (net 8))
   (segment (start 159.15 100.376) (end 159.131 100.395) (width 0.25) (layer "F.Cu") (net 8))
-  (segment (start 156.25 100.75) (end 156.7 100.3) (width 0.25) (layer "F.Cu") (net 8))
-  (segment (start 154.65 100.75) (end 156.25 100.75) (width 0.25) (layer "F.Cu") (net 8))
-  (segment (start 156.7 100.3) (end 156.7 99.05) (width 0.25) (layer "F.Cu") (net 8))
+  (segment (start 156.7 100.65) (end 156.7 99.05) (width 0.25) (layer "F.Cu") (net 8))
   (segment (start 159.15 99.25) (end 159.15 100.376) (width 0.25) (layer "F.Cu") (net 8))
   (segment (start 108.533122 106.2205) (end 107.188 106.2205) (width 1) (layer "F.Cu") (net 9))

Commit message: updated
Parts:
- removed Q5: MMBT5401, Package_TO_SOT_SMD:SOT-23
- removed Q6, Q7: SI2305A, Package_TO_SOT_SMD:SOT-23
- removed the R8 at (152.2, 74.3)
- removed the R8 at (152.2, 76.4)
- ? (x4): footprint MountingHole:MountingHole_3.2mm_M3_Pad_Via -> MountingHole:MountingHole_2.5mm
- moved C2 3.37 mm to (164.3, 91.1), turned to 90 degrees
- moved C3 3.17 mm to (162.1, 91.1), turned to 90 degrees
- moved D6 0.22 mm to (154.5, 105.6)
Connections:
- C1 pad 1: HATDC_5V -> BUCK_OUT
- C3 pad 1: HATDC_5V -> BUCK_OUT
- J4 pad 2: HATDC_5V -> BUCK_OUT
- J4 pad 4: HATDC_5V -> BUCK_OUT
- J8 pad 1: HATDC_5V -> BUCK_OUT
- J9 pad 1: HATDC_5V -> BUCK_OUT
- USB1 pad 1: HATDC_5V -> BUCK_OUT
- USB1 pad 5: HATDC_5V -> BUCK_OUT
Routing:
- net HATDC_5V: track 141.4 -> 0.00 mm, vias 8 -> 0
- net BUCK_OUT: track 22.2 -> 148.4 mm, vias 0 -> 8
- net BUCK_IN: track 134.0 -> 117.4 mm
- net Net-(Q6-Pad1): track 7.51 -> 0.00 mm
- net Net-(Q5-Pad1): track 4.16 -> 0.00 mm
- net GND: vias 7 -> 6
- removed copper zone on F.Cu, net HATDC_5V
Other:
- board text added: "Orange Juice v0.6 Design by Jerry for klipper B站：大石头Jerry"
- board text removed: "Orange Juice v0.5 Design by Jerry for klipper B站：大石头Jerry"

Commit message: Official v0.6 release
Parts:
- R19: value 4.7K -> 4K7

Commit message: update to v0.7
Parts:
- moved J7 0.09 mm to (144.1, 99.2)
- moved Q3 0.07 mm to (103.5, 105.3)
- moved Q4 0.07 mm to (99.7, 105.3)
Connections:
- net USB_DM2 renamed USB2_D-
- net USB_DM3 renamed USB3_D-
- net USB_DP2 renamed USB2_D+
- net USB_DP3 renamed USB3_D+
Routing:
- net BUCK_IN: track 117.4 -> 119.5 mm
- net USB2_D+: track 19.9 -> 21.6 mm
- net USB3_D-: track 32.8 -> 31.9 mm
- net USB3_D+: track 32.7 -> 33.4 mm
- net USB2_D-: track 19.8 -> 20.5 mm

Commit message: update to v0.7
Parts:
- removed the C1 at (156.9, 72.1)
- removed the C1 at (153.4, 95.0)
- removed the C3 at (162.1, 91.1)
- removed the C3 at (156.9, 74.2)
- removed C5: 22uF, Capacitor_SMD:C_0805_2012Metric
- removed C6: 0.1uF, Capacitor_SMD:C_0805_2012Metric
- removed C7: 33pF, Capacitor_SMD:C_0805_2012Metric
- removed D1: 10v, Diode_SMD:D_SOD-123
- removed the D2 at (167.8, 111.2)
- removed J13: FAN_12/24v, Connector_JST:JST_XH_B2B-XH-A_1x02_P2.50mm_Vertical
- removed Q1: AO4407A, JerryLibrary:SOIC127P600X175-8N
- removed R1: 100K, Resistor_SMD:R_0805_2012Metric
- removed R19: 4K7, Resistor_SMD:R_0805_2012Metric
- removed the R6 at (153.4, 92.9)
- removed the R8 at (153.4, 99.1)
- removed the R9 at (157.0, 97.0)
- added ?: GPIO6_Head, Connector_PinHeader_2.54mm:PinHeader_1x03_P2.54mm_Vertical, F.Cu at (91.7, 97.3)
- added ?: GPIO12_Head, Connector_PinHeader_2.54mm:PinHeader_1x03_P2.54mm_Vertical, F.Cu at (91.7, 104.9)
- added ?: GPIO11_Head, Connector_PinHeader_2.54mm:PinHeader_1x03_P2.54mm_Vertical, F.Cu at (91.7, 101.1)
- added C1: 10uF, Capacitor_SMD:C_1206_3216Metric, F.Cu at (161.3, 98.7)
- added C3: 10nF, Capacitor_SMD:C_0805_2012Metric, F.Cu at (167.6, 90.0)
- added D3: PWM2_STATUS, LED_SMD:LED_0805_2012Metric, F.Cu at (167.6, 113.3)
- added D5: B340A, Diode_SMD:D_SMA, F.Cu at (166.9, 94.7)
- added U2: TPS5430DDA, Package_SO:TI_SO-PowerPAD-8_ThermalVias, F.Cu at (162.2, 93.5)
- added U3: USBLC6-2SC6, Package_TO_SOT_SMD:SOT-23-6, F.Cu at (155.6, 72.1)
- C2: value 22uF -> 10uF
- C4: value 22uF -> 220uF; footprint Capacitor_SMD:C_0805_2012Metric -> Capacitor_SMD:C_Elec_6.3x5.4
- D6: footprint Diode_SMD:D_SMB -> Diode_SMD:D_SMA
- L1: value 4.7uH -> 22uH; footprint Inductor_SMD:L_Abracon_ASPI-0630LR -> Inductor_SMD:L_7.3x7.3_H4.5
- R2: value 9.09K -> 100K
- R3: value 100K -> 25K
- R4: value 10 -> 10K
- R5: value 100K -> 3.24K
- R7: value 20K -> 4k7
- U1: value MP2315GJ-Z -> USBLC6-2SC6; footprint Package_TO_SOT_SMD:SOT-23-8 -> Package_TO_SOT_SMD:SOT-23-6
- moved U1 23.2 mm to (155.6, 68.5), turned to 0 degrees
- moved J8 21.4 mm to (112.8, 112.8), turned to 180 degrees
- moved R7 18.1 mm to (167.6, 109.6), turned to -90 degrees
- moved C2 10.6 mm to (161.3, 101.2), turned to 180 degrees
- moved J12 10.4 mm to (134.4, 112.8)
- moved R4 10.4 mm to (143.7, 107.7)
- moved D3 10.4 mm to (131.6, 107.7)
- moved D4 10.4 mm to (122.4, 107.7)
- moved R10 10.4 mm to (126.0, 107.7)
- moved J15 10.4 mm to (125.5, 112.8)
- moved D2 10.4 mm to (140.2, 107.7)
- moved J10 10.4 mm to (143.3, 112.8)
- moved R7 10.4 mm to (135.1, 107.7)
- moved R5 8.40 mm to (158.2, 94.2), turned to -90 degrees
- moved R3 7.32 mm to (156.6, 97.5), turned to 180 degrees
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Connections:
- D6 pad 1: DC_IN -> BUCK_IN
- J11 pad 1: UART1_RX -> UART1_TX
- J11 pad 2: UART1_TX -> UART1_RX
- J2 pad 1: DC_IN -> GND
- J2 pad 2: GND -> BUCK_IN
- J4 pad 10: UART1_TX -> UART1_RX
- J4 pad 3: unconnected-(J2-Pad3) -> GPIO12
- J4 pad 5: unconnected-(J2-Pad5) -> GPIO11
- J4 pad 7: unconnected-(J2-Pad7) -> GPIO6
- J4 pad 8: UART1_RX -> UART1_TX
- L1 pad 1: BUCK_SW -> BUCK_PH
- R2 pad 1: GND -> BUCK_IN
- R2 pad 2: BUCK_AAM -> BUCK_EN
- R3 pad 1: BUCK_IN -> BUCK_EN
- R3 pad 2: BUCK_EN -> GND
- R4 pad 1: BUCK_BST -> BUCK_OUT
- R4 pad 2: Net-(C6-Pad1) -> BUCK_VSNS
- R5 pad 1: Net-(D1-Pad2) (its old number) -> BUCK_VSNS
- R7 pad 1: BUCK_FB -> BUCK_IN
- U1 pad 1: BUCK_AAM -> USB2_D-
- U1 pad 2: BUCK_IN -> GND
- U1 pad 3: BUCK_SW -> USB2_D+
- U1 pad 4: GND -> USB2_Conn_D+
- U1 pad 5: BUCK_BST -> BUCK_OUT
- U1 pad 6: BUCK_EN -> USB2_Conn_D-
- USB1 pad 2: USB2_D- -> USB2_Conn_D-
- USB1 pad 3: USB2_D+ -> USB2_Conn_D+
- USB1 pad 6: USB3_D- -> USB3_Conn_D-
- USB1 pad 7: USB3_D+ -> USB3_Conn_D+
Routing:
- net BUCK_IN: track 119.5 -> 94.4 mm, vias 10 -> 0
- net USB3_D+: track 33.4 -> 17.5 mm
- net USB3_D-: track 31.9 -> 17.5 mm, vias 1 -> 0
- net GPIO12: track 0.00 -> 11.6 mm
- net Net-(C1-Pad1): track 11.1 -> 0.00 mm
- net GPIO11: track 0.00 -> 10.3 mm
- net Net-(D2-Pad1): track 30.2 -> 39.6 mm
- net GPIO6: track 0.00 -> 9.37 mm
- net USB3_Conn_D+: track 0.00 -> 8.63 mm, vias 0 -> 1
- net Net-(D3-Pad1): track 25.6 -> 34.0 mm
- net Net-(D1-Pad2) (its old number): track 7.75 -> 0.00 mm
- net USB3_Conn_D-: track 0.00 -> 7.51 mm
- net BUCK_OUT: track 148.6 -> 156.1 mm, vias 8 -> 10
- net Net-(D4-Pad1): track 20.4 -> 27.2 mm
- net USB2_Conn_D-: track 0.00 -> 5.90 mm
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- added copper zone on F.Cu, net BUCK_PH
- removed copper zone on F.Cu, net BUCK_SW
- removed copper zone on F.Cu, net DC_IN
Other:
- board text added: "-"
- board text added: "12/24V"
- board text added: "5v"
- board text added: "DC 5V"
- board text added: "GPIO11"
- board text added: "GPIO12"
- board text added: "GPIO6"
- board text added: "Orange Juice v0.7 Design by Jerry for klipper B站：大石头Jerry"
- board text removed: "DC 12/24V"
- board text removed: "Orange Juice v0.6 Design by Jerry for klipper B站：大石头Jerry"

Commit message: update to v0.7
Parts:
- L1: footprint Inductor_SMD:L_7.3x7.3_H4.5 -> Inductor_SMD:L_Abracon_ASPI-0630LR
- gave numbers to parts that had none: 3
Routing:
- net BUCK_OUT: track 156.1 -> 158.8 mm

Commit message: update to v0.7
Parts:
- moved J12 0.15 mm to (148.8, 83.7)
Changed lines of the file:
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@@
     (fp_line (start 3.7 -3.4) (end -3.7 -3.4) (layer "F.SilkS") (width 0.12))
     (fp_line (start 3.7 3.4) (end 3.7 1.9) (layer "F.SilkS") (width 0.12))
+    (fp_line (start 4.45 1.95) (end 4.45 -1.95) (layer "F.CrtYd") (width 0.05))
+    (fp_line (start 3.85 1.95) (end 4.45 1.95) (layer "F.CrtYd") (width 0.05))
+    (fp_line (start 3.85 -3.58) (end -3.85 -3.58) (layer "F.CrtYd") (width 0.05))
+    (fp_line (start -3.85 1.95) (end -3.85 3.58) (layer "F.CrtYd") (width 0.05))
+    (fp_line (start -4.45 1.95) (end -3.85 1.95) (layer "F.CrtYd") (width 0.05))
+    (fp_line (start -4.45 -1.95) (end -4.45 1.95) (layer "F.CrtYd") (width 0.05))
+    (fp_line (start 4.45 -1.95) (end 3.85 -1.95) (layer "F.CrtYd") (width 0.05))
+    (fp_line (start -3.85 -1.95) (end -4.45 -1.95) (layer "F.CrtYd") (width 0.05))
+    (fp_line (start 3.85 3.58) (end 3.85 1.95) (layer "F.CrtYd") (width 0.05))
+    (fp_line (start -3.85 3.58) (end 3.85 3.58) (layer "F.CrtYd") (width 0.05))
     (fp_line (start 3.85 -1.95) (end 3.85 -3.58) (layer "F.CrtYd") (width 0.05))
-    (fp_line (start 3.85 -3.58) (end -3.85 -3.58) (layer "F.CrtYd") (width 0.05))
-    (fp_line (start 4.45 1.95) (end 4.45 -1.95) (layer "F.CrtYd") (width 0.05))
     (fp_line (start -3.85 -3.58) (end -3.85 -1.95) (layer "F.CrtYd") (width 0.05))
-    (fp_line (start -4.45 1.95) (end -3.85 1.95) (layer "F.CrtYd") (width 0.05))
-    (fp_line (start -3.85 3.58) (end 3.85 3.58) (layer "F.CrtYd") (width 0.05))
-    (fp_line (start 3.85 3.58) (end 3.85 1.95) (layer "F.CrtYd") (width 0.05))
-    (fp_line (start -3.85 -1.95) (end -4.45 -1.95) (layer "F.CrtYd") (width 0.05))
-    (fp_line (start 4.45 -1.95) (end 3.85 -1.95) (layer "F.CrtYd") (width 0.05))
-    (fp_line (start -3.85 1.95) (end -3.85 3.58) (layer "F.CrtYd") (width 0.05))
-    (fp_line (start 3.85 1.95) (end 4.45 1.95) (layer "F.CrtYd") (width 0.05))
-    (fp_line (start -4.45 -1.95) (end -4.45 1.95) (layer "F.CrtYd") (width 0.05))
     (fp_line (start 3.6 3.325) (end -3.6 3.325) (layer "F.Fab") (width 0.1))
     (fp_line (start -3.6 3.325) (end -3.6 -3.325) (layer "F.Fab") (width 0.1))
@@
   )
   (footprint "Connector_PinSocket_2.54mm:PinSocket_1x08_P2.54mm_Vertical" locked (layer "F.Cu")
-    (at 148.925 83.725)
+    (at 148.775 83.725)
     (descr "Through hole straight socket strip, 1x08, 2.54mm pitch, single row (from Kicad 4.0.7), script generated")
     (tags "Through hole socket strip THT 1x08 2.54mm single row")
