File: kicad/orange_juice_board.kicad_pcb (KiCad board)
At the start: 2 copper layers, 85 x 56 mm, 56 parts, among them J10 GPIO12_Head, J10 PWM_OUT1, J11 CONN_UART, J12 Conn_01x08, J12 PWM_OUT2, J13 GPIO6_Head, J14 GPIO11_Head, J15 PWM_OUT3, J2 DC_INPUT, J3 CONN_ADXL345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

Commit message: minor update
Parts:
- moved C3 0.72 mm to (166.9, 89.9)
- moved J12 0.25 mm to (149.0, 83.7)
Routing:
- net BUCK_BOOT: track 2.86 -> 2.31 mm

Commit message: update bom
Parts:
- R3: value 25K -> 25K5
Changed lines of the file:
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@@
     (descr "Diode SMA (DO-214AC)")
     (tags "Diode SMA (DO-214AC)")
+    (property "LCSC Part#" "C64982")
     (property "Sheetfile" "orange_juice_board.kicad_sch")
     (property "Sheetname" "")
@@
     (descr "SMD capacitor, aluminum electrolytic nonpolar, 6.3x5.4mm")
     (tags "capacitor electrolyic nonpolar")
+    (property "LCSC Part#" "C3345")
     (property "Sheetfile" "orange_juice_board.kicad_sch")
     (property "Sheetname" "")
@@
     (descr "Capacitor SMD 0805 (2012 Metric), square (rectangular) end terminal, IPC_7351 nominal, (Body size source: IPC-SM-782 page 76, https://www.pcb-3d.com/wordpress/wp-content/uploads/ipc-sm-782a_amendment_1_and_2.pdf, https://docs.google.com/spreadsheets/d/1BsfQQcO9C6DZCsRaXUlFlo91Tg2WpOkGARC1WS5S8t0/edit?usp=sharing), generated with kicad-footprint-generator")
     (tags "capacitor")
+    (property "LCSC Part#" "C83170")
     (property "Sheetfile" "orange_juice_board.kicad_sch")
     (property "Sheetname" "")
@@
     (descr "Resistor SMD 0805 (2012 Metric), square (rectangular) end terminal, IPC_7351 nominal, (Body size source: IPC-SM-782 page 72, https://www.pcb-3d.com/wordpress/wp-content/uploads/ipc-sm-782a_amendment_1_and_2.pdf), generated with kicad-footprint-generator")
     (tags "resistor")
+    (property "LCSC Part#" "C84376")
     (property "Sheetfile" "orange_juice_board.kicad_sch")
     (property "Sheetname" "")
@@
     (descr "8-pin HTSOP package with 1.27mm pin pitch, compatible with SOIC-8, 3.9x4.9mm² body, exposed pad, thermal vias with large copper area, as proposed in http://www.ti.com/lit/ds/symlink/tps5430.pdf")
     (tags "HTSOP 1.27")
+    (property "LCSC Part#" "C9864")
     (property "Sheetfile" "orange_juice_board.kicad_sch")
     (property "Sheetname" "")
@@
     (descr "Resistor SMD 0805 (2012 Metric), square (rectangular) end terminal, IPC_7351 nominal, (Body size source: IPC-SM-782 page 72, https://www.pcb-3d.com/wordpress/wp-content/uploads/ipc-sm-782a_amendment_1_and_2.pdf), generated with kicad-footprint-generator")
     (tags "resistor")
+    (property "LCSC Part#" "C100049")
     (property "Sheetfile" "orange_juice_board.kicad_sch")
     (property "Sheetname" "")
@@
     (descr "SOT, 6 Pin (https://www.jedec.org/sites/default/files/docs/Mo-178c.PDF variant AB), generated with kicad-footprint-generator ipc_gullwing_generator.py")
     (tags "SOT TO_SOT_SMD")
+    (property "LCSC Part#" "C2687116")
     (property "Sheetfile" "orange_juice_board.kicad_sch")
     (property "Sheetname" "")
@@
     (descr "smd shielded power inductor https://abracon.com/Magnetics/power/ASPI-0630LR.pdf")
     (tags "inductor abracon smd shielded")
+    (property "LCSC Part#" "C128694")
     (property "Sheetfile" "orange_juice_board.kicad_sch")
     (property "Sheetname" "")
@@
     (descr "Resistor SMD 0805 (2012 Metric), square (rectangular) end terminal, IPC_7351 nominal, (Body size source: IPC-SM-782 page 72, https://www.pcb-3d.com/wordpress/wp-content/uploads/ipc-sm-782a_amendment_1_and_2.pdf), generated with kicad-footprint-generator")
     (tags "resistor")
+    (property "LCSC Part#" "C228665")
     (property "Sheetfile" "orange_juice_board.kicad_sch")
     (property "Sheetname" "")
@@
       (effects (font (size 1 1) (thickness 0.15)))
     )
-    (fp_text value "25K" (at 0 1.65) (layer "F.Fab")
+    (fp_text value "25K5" (at 0 1.65) (layer "F.Fab")
       (effects (font (size 1 1) (thickness 0.15)))
     )
@@
     (descr "Resistor SMD 0805 (2012 Metric), square (rectangular) end terminal, IPC_7351 nominal, (Body size source: IPC-SM-782 page 72, https://www.pcb-3d.com/wordpress/wp-content/uploads/ipc-sm-782a_amendment_1_and_2.pdf), generated with kicad-footprint-generator")
     (tags "resistor")
+    (property "LCSC Part#" "C273976")
     (property "Sheetfile" "orange_juice_board.kicad_sch")
     (property "Sheetname" "")
@@
     (descr "Capacitor SMD 1206 (3216 Metric), square (rectangular) end terminal, IPC_7351 nominal, (Body size source: IPC-SM-782 page 76, https://www.pcb-3d.com/wordpress/wp-content/uploads/ipc-sm-782a_amendment_1_and_2.pdf), generated with kicad-footprint-generator")
     (tags "capacitor")
+    (property "LCSC Part#" "C723460")
     (property "Sheetfile" "orange_juice_board.kicad_sch")
     (property "Sheetname" "")
@@
     (descr "Capacitor SMD 1206 (3216 Metric), square (rectangular) end terminal, IPC_7351 nominal, (Body size source: IPC-SM-782 page 76, https://www.pcb-3d.com/wordpress/wp-content/uploads/ipc-sm-782a_amendment_1_and_2.pdf), generated with kicad-footprint-generator")
     (tags "capacitor")
+    (property "LCSC Part#" "C723460")
     (property "Sheetfile" "orange_juice_board.kicad_sch")
     (property "Sheetname" "")
@@
     (descr "SOT, 6 Pin (https://www.jedec.org/sites/default/files/docs/Mo-178c.PDF variant AB), generated with kicad-footprint-generator ipc_gullwing_generator.py")
     (tags "SOT TO_SOT_SMD")
-    (property "Sheetfile" "orange_juice_board.kicad_sch")
-    (property "Sheetname" "")
+    (property "LCSC Part#" "C2687116")
+    (property "Sheetfile" "orange_juice_board.kicad_sch")
+    (property "Sheetname" "")
