File: kicad/orange_juice_board.kicad_sch (KiCad schematic)
At the start: 54 parts, among them J10 PWM_OUT1, J11 CONN_UART, J12 PWM_OUT2, J13 FAN_12/24v, J15 PWM_OUT3, J2 DC_INPUT, J3 CONN_ADXL345, J4 OrangePi Zero GPIO PINs, J5 Conn_MAX31865, J7 OrangePi Zero Function Interf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, J8 FAN_5v, J9 PWR_5v, Q1 AO3401A, Q2 AO3400A, Q3 AO3400A, Q4 AO3400A, U1 TPS5430

Commit message: update version 0.3
Parts:
- renumbered D5 to D4, D4 to D5
Connections:
- net GND: no longer USB1.9 (Shield)
Other:
- moved on the sheet: D2, D3, D4

Commit message: bate version
Parts:
- removed C2: 10u, Capacitor_SMD:C_1206_3216Metric, symbol orange_juice_board-rescue:C_Small-Device-OrangePiZeroExtentionBoard-rescue-oran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
- removed C4: 10n, Capacitor_SMD:C_0805_2012Metric, symbol orange_juice_board-rescue:C_Small-Device-OrangePiZeroExtentionBoard-rescue-oran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
- removed C5: 220u, Capacitor_SMD:CP_Elec_6.3x5.4, symbol orange_juice_board-rescue:CP1_Small-Device-OrangePiZeroExtentionBoard-rescue-or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
- removed D1: PWR_LED, LED_SMD:LED_0805_2012Metric, symbol orange_juice_board-rescue:LED_Small-Device-OrangePiZeroExtentionBoard-rescue-or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
- removed D5: B340A, Diode_SMD:D_SMA, symbol orange_juice_board-rescue:B340-Diode-OrangePiZeroExtentionBoard-rescue-orange_j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
- removed L1: 15u, Inductor_SMD:L_Sumida_CDMC6D28_7.25x6.5mm, symbol orange_juice_board-rescue:L_Small-Device-OrangePiZeroExtentionBoard-rescue-oran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
- removed Q1: AO3401A, Package_TO_SOT_SMD:SOT-23, symbol orange_juice_board-rescue:AO3401A-Transistor_FET-OrangePiZeroExtentionBoard-res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
- removed R1: 4k7, Resistor_SMD:R_0805_2012Metric, symbol orange_juice_board-rescue:R_Small-Device-OrangePiZeroExtentionBoard-rescue-oran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
- removed R11: 10k, Resistor_SMD:R_0805_2012Metric, symbol orange_juice_board-rescue:R_Small-Device-OrangePiZeroExtentionBoard-rescue-oran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
- removed R12: 3k, Resistor_SMD:R_0805_2012Metric, symbol orange_juice_board-rescue:R_Small-Device-OrangePiZeroExtentionBoard-rescue-oran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
- removed R13: 240, Resistor_SMD:R_0805_2012Metric, symbol orange_juice_board-rescue:R_Small-Device-OrangePiZeroExtentionBoard-rescue-oran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
- removed R2: 100k, Resistor_SMD:R_0805_2012Metric, symbol orange_juice_board-rescue:R_Small-Device-OrangePiZeroExtentionBoard-rescue-oran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
- removed R3: 21k, Resistor_SMD:R_0805_2012Metric, symbol orange_juice_board-rescue:R_Small-Device-OrangePiZeroExtentionBoard-rescue-oran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
- removed U1: TPS5430, Package_SO:TI_SO-PowerPAD-8_ThermalVias, symbol orange_juice_board-rescue:TPS5430DDA-Regulator_Switching-OrangePiZeroExtentionB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
- added C1, C3, C6: 0.1uF, Capacitor_SMD:C_0805_2012Metric, symbol Device:C_Small
- added C2: 22uF, Capacitor_SMD:C_1206_3216Metric, symbol Device:C_Small
- added C4, C5: 22uF, Capacitor_SMD:C_0805_2012Metric, symbol Device:C_Small
- added C7: 33pF, Capacitor_SMD:C_0805_2012Metric, symbol Device:C_Small
- added D1: 10v, Diode_SMD:D_SOD-123, symbol Device:D_Zener_Small
- added D2: PWM1_STATUS, LED_SMD:LED_0805_2012Metric, symbol orange_juice_board-rescue:LED_Small-Device-OrangePiZeroExtentionBoard-rescue-or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
- added L1: 4.7uH, Inductor_SMD:L_Abracon_ASPI-0630LR, symbol Device:L_Small
- added Q1: AO4407A, JerryLibrary:SOIC127P600X175-8N, symbol Device:Q_PMOS_SGD
- added R1, R3, R5: 100K, Resistor_SMD:R_0805_2012Metric, symbol Device:R_Small
- added R19: 4.7K, Resistor_SMD:R_0805_2012Metric, symbol Device:R_Small
- added R2: 9.09K, Resistor_SMD:R_0805_2012Metric, symbol Device:R_Small
- added R4: 10, Resistor_SMD:R_0805_2012Metric, symbol Device:R_Small
- added R6: 16.9K, Resistor_SMD:R_0805_2012Metric, symbol Device:R_Small
- added R7: 20K, Resistor_SMD:R_0805_2012Metric, symbol Device:R_Small
- added R8: 40.2K, Resistor_SMD:R_0805_2012Metric, symbol Device:R_Small
- added R9: 7.5K, Resistor_SMD:R_0805_2012Metric, symbol Device:R_Small
- added U1: MP2315GJ-Z, Package_TO_SOT_SMD:SOT-23-8, symbol Jerry_Library:MP2315GJ-Z
Connections:
- net +5V: now also C4.1, C5.1, C7.2, L1.2, R8.2; no longer J7.13 (Pin_13)
- net BUCK_EN: now also R3.2, R6.1, U1.6 (EN/SYNC)
- net BUCK_IN: now also J10.1 (Pin_1), J12.1 (Pin_1), J13.1 (Pin_1), J15.1 (Pin_1), R10.2, R4.2, R7.2, C2.1, C3.1, D1.1 (K), Q1.1 (S), R19.1, R3.1, U1.2 (IN)
- net GND: now also C1.2, C2.2, C3.2, C4.2, C5.2, D2.1 (K), R2.1, R5.2, R6.2, R9.1, U1.4 (GND)
- removed net DCIN: J10.1 (Pin_1), J12.1 (Pin_1), J13.1 (Pin_1), J15.1 (Pin_1), J2.1 (Pin_1), R10.2, R4.2, R7.2
- new net: C7.1, R7.2, R8.1, R9.2
- new net: D2.2 (A), R19.2
- new net: C6.1, R4.2
- new net: D1.2 (A), Q1.2 (G), R5.1
- new net: C1.1, R1.2, U1.7 (VCC)
- new net BUCK_AAM: R1.1, R2.2, U1.1 (AAM)
- new net BUCK_BST: R4.1, U1.5 (BST)
- new net BUCK_FB: R7.1, U1.8 (FB)
- new net BUCK_SW: C6.2, L1.1, U1.3 (SW)
- new net DC_IN: J2.1 (Pin_1), Q1.3 (D)
- no-connect marks 12 -> 13
Other:
- note added: "5V"
- moved on the sheet: J10, J12, J13, J15

Commit message: update v0.6
Parts:
- removed J5: Conn_MAX31865, Connector_PinSocket_2.54mm:PinSocket_1x06_P2.54mm_Vertical, symbol orange_juice_board-rescue:Conn_01x06-Connector_Generic-OrangePiZeroExtentionBoa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
- added D6: D_TVS, Diode_SMD:D_SMB, symbol Device:D_TVS
- added J12: Conn_01x08, Connector_PinSocket_2.54mm:PinSocket_1x08_P2.54mm_Vertical, symbol Connector_Generic:Conn_01x08
- added Q5: MMBT5401, Package_TO_SOT_SMD:SOT-23, symbol Device:Q_PMOS_GSD
- added Q6, Q7: SI2305A, Package_TO_SOT_SMD:SOT-23, symbol Device:Q_PNP_CBE
- added R8 (x2): 100, Resistor_SMD:R_0805_2012Metric, symbol orange_juice_board-rescue:R_Small-Device-OrangePiZeroExtentionBoard-rescue-oran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
Connections:
- net DC_IN: now also D6.2 (A2)
- net GND: now also D6.1 (A1), J12.2 (Pin_2), R8.2, R8.2
- net GPIO_0_SDI: now also J12.6 (Pin_6)
- net GPIO_1_CS: now also J12.7 (Pin_7)
- net GPIO_2_CLK: now also J12.4 (Pin_4)
- net GPIO_3_SDO: now also J12.5 (Pin_5)
- net +3V3 renamed PI_3.3V
- net PI_3.3V: now also J12.3 (Pin_3)
- net +5V renamed HATDC_5V
- net HATDC_5V: now also Q5.3 (D), Q6.3 (E); no longer C4.1, C5.1, C7.2, L1.2, R8.2
- new net: Q6.1 (C), Q6.2 (B), Q7.2 (B), R8.1
- new net: Q5.1 (G), Q7.1 (C), R8.1
- new net BUCK_OUT: C4.1, C5.1, C7.2, L1.2, Q5.2 (S), Q7.3 (E), R8.2
- no-connect marks 13 -> 15
Other:
- company: Stone-Jerry -> Stone Lab - Jerry
- title: Orange Pi Zero Adapter -> Orange Juice
- moved on the sheet: C1, C3, D2, D3, D4, H10, H5, H6, H7, H8, H9, J10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

Commit message: update to v0.6
Parts:
- D6: value D_TVS -> SMAJ24A; symbol Device:D_TVS -> Diode:SM6T24A
Connections:
- net DC_IN: now also D6.1 (A1); no longer D6.2 (A2)
- net GND: now also D6.2 (A2); no longer D6.1 (A1)
Changed lines of the file:
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@@
     (pin "1")
   )
-  (symbol (lib_id "Device:D_TVS") (at 34.29 43.18 90) (unit 1)
-    (in_bom yes) (on_board yes) (fields_autoplaced)
-    (property "Reference" "D6" (id 0) (at 36.83 41.9099 90)
-      (effects (font (size 1.27 1.27)) (justify right))
-    )
-    (property "Value" "D_TVS" (id 1) (at 36.83 44.4499 90)
-      (effects (font (size 1.27 1.27)) (justify right))
-    )
-    (property "Footprint" "Diode_SMD:D_SMB" (id 2) (at 34.29 43.18 0)
-      (effects (font (size 1.27 1.27)) hide)
-    )
-    (property "Datasheet" "~" (id 3) (at 34.29 43.18 0)
+  (symbol (lib_id "Diode:SM6T24A") (at 34.29 43.18 270) (unit 1)
+    (in_bom yes) (on_board yes)
+    (property "Reference" "D6" (id 0) (at 27.94 41.91 90)
+      (effects (font (size 1.27 1.27)) (justify left))
+    )
+    (property "Value" "SMAJ24A" (id 1) (at 24.13 44.45 90)
+      (effects (font (size 1.27 1.27)) (justify left))
+    )
+    (property "Footprint" "Diode_SMD:D_SMB" (id 2) (at 29.21 43.18 0)
+      (effects (font (size 1.27 1.27)) hide)
+    )
+    (property "Datasheet" "https://www.st.com/resource/en/datasheet/sm6t.pdf" (id 3) (at 34.29 41.91 0)
       (effects (font (size 1.27 1.27)) hide)
     )
@@
     )
     (path "/c909aa0c-2fd9-4d9c-a4ea-3fb1adec5ed8"
-      (reference "D6") (unit 1) (value "D_TVS") (footprint "Diode_SMD:D_SMB")
+      (reference "D6") (unit 1) (value "SMAJ24A") (footprint "Diode_SMD:D_SMB")
     )
     (path "/00000000-0000-0000-0000-000061cd640e"

Commit message: updated
Parts:
- removed Q5: MMBT5401, Package_TO_SOT_SMD:SOT-23, symbol Device:Q_PMOS_GSD
- removed Q6, Q7: SI2305A, Package_TO_SOT_SMD:SOT-23, symbol Device:Q_PNP_CBE
- removed R8 (x2): 100, Resistor_SMD:R_0805_2012Metric, symbol orange_juice_board-rescue:R_Small-Device-OrangePiZeroExtentionBoard-rescue-oran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
Connections:
- net HATDC_5V is gone; now on net BUCK_OUT: C1.1, C3.1, J4.2 (Pin_2), J4.4 (Pin_4), J8.1 (Pin_1), J9.1 (Pin_1), USB1.1 (VCC), USB1.5 (VCC)
Other:
- moved on the sheet: D2, D3, D4, J10, J11, J12, J13, J15, Q2, Q3, Q4, R10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

Commit message: Official v0.6 release
Parts:
- C1, C3, C6: LCSC Part# (none) -> C49678
- C2: LCSC Part# (none) -> C2835562
- C4, C5: LCSC Part# (none) -> C29277
- C7: LCSC Part# (none) -> C107115
- D1: LCSC Part# (none) -> C21564
- D6: LCSC Part# (none) -> C726750
- L1: LCSC Part# (none) -> C128688
- Q1: LCSC Part# (none) -> C557949
- R1, R3, R5: LCSC Part# (none) -> C96346
- R19: value 4.7K -> 4K7; LCSC Part# (none) -> C60816
- R2: LCSC Part# (none) -> C17854
- R4: LCSC Part# (none) -> C17415
- R6: LCSC Part# (none) -> C228334
- R7: LCSC Part# (none) -> C229162
- R8: LCSC Part# (none) -> C228820
- R9: LCSC Part# (none) -> C114547
Changed lines of the file:
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@@
     (in_bom yes) (on_board yes)
     (property "Reference" "R16" (id 0) (at 153.67 111.76 90))
-    (property "Value" "10k" (id 1) (at 153.67 116.84 90))
+    (property "Value" "10K" (id 1) (at 153.67 116.84 90))
     (property "Footprint" "Resistor_SMD:R_0805_2012Metric" (id 2) (at 153.67 114.3 0)
       (effects (font (size 1.27 1.27)) hide)
@@
     (in_bom yes) (on_board yes)
     (property "Reference" "R17" (id 0) (at 205.74 111.76 90))
-    (property "Value" "10k" (id 1) (at 205.74 116.84 90))
+    (property "Value" "10K" (id 1) (at 205.74 116.84 90))
     (property "Footprint" "Resistor_SMD:R_0805_2012Metric" (id 2) (at 205.74 114.3 0)
       (effects (font (size 1.27 1.27)) hide)
@@
     (in_bom yes) (on_board yes)
     (property "Reference" "R18" (id 0) (at 259.08 111.76 90))
-    (property "Value" "10k" (id 1) (at 259.08 116.84 90))
+    (property "Value" "10K" (id 1) (at 259.08 116.84 90))
     (property "Footprint" "Resistor_SMD:R_0805_2012Metric" (id 2) (at 259.08 114.3 0)
       (effects (font (size 1.27 1.27)) hide)
@@
     (in_bom yes) (on_board yes)
     (property "Reference" "C8" (id 0) (at 35.56 161.29 90))
-    (property "Value" "22u" (id 1) (at 35.56 168.6052 90))
+    (property "Value" "22uF" (id 1) (at 35.56 168.6052 90))
     (property "Footprint" "Capacitor_SMD:C_0805_2012Metric" (id 2) (at 35.56 165.1 0)
       (effects (font (size 1.27 1.27)) hide)
@@
     (in_bom yes) (on_board yes)
     (property "Reference" "C9" (id 0) (at 71.12 159.2834 90))
-    (property "Value" "22u" (id 1) (at 71.12 161.5948 90))
+    (property "Value" "22uF" (id 1) (at 71.12 161.5948 90))
     (property "Footprint" "Capacitor_SMD:C_0805_2012Metric" (id 2) (at 71.12 165.1 0)
       (effects (font (size 1.27 1.27)) hide)
@@
     (in_bom yes) (on_board yes)
     (property "Reference" "R10" (id 0) (at 135.89 81.3816 90))
-    (property "Value" "4k7" (id 1) (at 135.89 83.693 90))
+    (property "Value" "4K7" (id 1) (at 135.89 83.693 90))
     (property "Footprint" "Resistor_SMD:R_0805_2012Metric" (id 2) (at 135.89 86.36 0)
       (effects (font (size 1.27 1.27)) hide)
@@
     (in_bom yes) (on_board yes)
     (property "Reference" "R11" (id 0) (at 187.96 81.3816 90))
-    (property "Value" "4k7" (id 1) (at 187.96 83.693 90))
+    (property "Value" "4K7" (id 1) (at 187.96 83.693 90))
     (property "Footprint" "Resistor_SMD:R_0805_2012Metric" (id 2) (at 187.96 86.36 0)
       (effects (font (size 1.27 1.27)) hide)
@@
     (in_bom yes) (on_board yes)
     (property "Reference" "R12" (id 0) (at 241.3 81.3816 90))
-    (property "Value" "4k7" (id 1) (at 241.3 83.693 90))
+    (property "Value" "4K7" (id 1) (at 241.3 83.693 90))
     (property "Footprint" "Resistor_SMD:R_0805_2012Metric" (id 2) (at 241.3 86.36 0)
       (effects (font (size 1.27 1.27)) hide)
@@
       (effects (font (size 1.27 1.27)) hide)
     )
+    (property "LCSC Part#" "C17854" (id 4) (at 130.81 31.75 0)
+      (effects (font (size 1.27 1.27)) hide)
+    )
     (pin "1")
     (pin "2")
@@
       (effects (font (size 1.27 1.27)) hide)
     )
+    (property "LCSC Part#" "C228820" (id 4) (at 243.84 58.42 0)
+      (effects (font (size 1.27 1.27)) hide)
+    )
     (pin "1")
     (pin "2")
@@
       (effects (font (size 1.27 1.27)) (justify left))
     )
-    (property "Value" "4.7K" (id 1) (at 63.5 35.5599 0)
+    (property "Value" "4K7" (id 1) (at 63.5 35.5599 0)
       (effects (font (size 1.27 1.27)) (justify left))
     )
@@
     )
     (property "Datasheet" "~" (id 3) (at 60.96 34.29 0)
+      (effects (font (size 1.27 1.27)) hide)
+    )
+    (property "LCSC Part#" "C60816" (id 4) (at 60.96 34.29 0)
       (effects (font (size 1.27 1.27)) hide)
     )
@@
       (effects (font (size 1.27 1.27)) hide)
     )
+    (property "LCSC Part#" "C2835562" (id 4) (at 72.39 34.29 0)
+      (effects (font (size 1.27 1.27)) hide)
+    )
     (pin "1")
     (pin "2")
@@
       (effects (font (size 1.27 1.27)) hide)
     )
+    (property "LCSC Part#" "C29277" (id 4) (at 260.35 34.29 0)
+      (effects (font (size 1.27 1.27)) hide)
+    )
     (pin "1")
     (pin "2")
@@
       (effects (font (size 1.27 1.27)) hide)
     )
+    (property "LCSC Part#" "C114547" (id 4) (at 238.76 63.5 0)
+      (effects (font (size 1.27 1.27)) hide)
+    )
     (pin "1")
     (pin "2")
@@
       (effects (font (size 1.27 1.27)) hide)
     )
+    (property "LCSC Part#" "C49678" (id 4) (at 237.49 38.1 0)
+      (effects (font (size 1.27 1.27)) hide)
+    )
     (pin "1")
     (pin "2")
@@
     )
     (property "Datasheet" "~" (id 3) (at 243.84 54.61 0)
+      (effects (font (size 1.27 1.27)) hide)
+    )
+    (property "LCSC Part#" "C107115" (id 4) (at 243.84 54.61 0)
       (effects (font (size 1.27 1.27)) hide)
     )
@@
       (effects (font (size 1.27 1.27)) hide)
     )
+    (property "LCSC Part#" "C557949" (id 4) (at 43.18 30.48 0)
+      (effects (font (size 1.27 1.27)) hide)
+    )
     (pin "1")
     (pin "2")
@@
       (effects (font (size 1.27 1.27)) hide)
     )
+    (property "LCSC Part#" "C49678" (id 4) (at 142.24 31.75 0)
+      (effects (font (size 1.27 1.27)) hide)
+    )
     (pin "1")
     (pin "2")
@@
     )
     (property "Datasheet" "~" (id 3) (at 43.18 43.18 0)
+      (effects (font (size 1.27 1.27)) hide)
+    )
+    (property "LCSC Part#" "C96346" (id 4) (at 43.18 43.18 0)
       (effects (font (size 1.27 1.27)) hide)
     )
@@
     )
     (property "Datasheet" "~" (id 3) (at 245.11 29.21 0)
+      (effects (font (size 1.27 1.27)) hide)
+    )
+    (property "LCSC Part#" "C128688" (id 4) (at 245.11 29.21 0)
       (effects (font (size 1.27 1.27)) hide)
     )
@@
       (effects (font (size 1.27 1.27)) hide)
     )
+    (property "LCSC Part#" "C96346" (id 4) (at 135.89 27.94 0)
+      (effects (font (size 1.27 1.27)) hide)
+    )
     (pin "1")
     (pin "2")
@@
       (effects (font (size 1.27 1.27)) hide)
     )
+    (property "LCSC Part#" "C726750" (id 4) (at 34.29 43.18 0)
+      (effects (font (size 1.27 1.27)) hide)
+    )
     (pin "1")
     (pin "2")
@@
       (effects (font (size 1.27 1.27)) hide)
     )
+    (property "LCSC Part#" "C29277" (id 4) (at 250.19 34.29 0)
+      (effects (font (size 1.27 1.27)) hide)
+    )
     (pin "1")
     (pin "2")
@@
       (effects (font (size 1.27 1.27)) hide)
     )
+    (property "LCSC Part#" "C49678" (id 4) (at 82.55 34.29 0)
+      (effects (font (size 1.27 1.27)) hide)
+    )
     (pin "1")
     (pin "2")
@@
       (effects (font (size 1.27 1.27)) hide)
     )
+    (property "LCSC Part#" "C228334" (id 4) (at 92.71 44.45 0)
+      (effects (font (size 1.27 1.27)) hide)
+    )
     (pin "1")
     (pin "2")
@@
       (effects (font (size 1.27 1.27)) hide)
     )
+    (property "LCSC Part#" "C229162" (id 4) (at 233.68 58.42 0)
+      (effects (font (size 1.27 1.27)) hide)
+    )
     (pin "1")
     (pin "2")
@@
       (effects (font (size 1.27 1.27)) hide)
     )
+    (property "LCSC Part#" "C17415" (id 4) (at 231.14 38.1 0)
+      (effects (font (size 1.27 1.27)) hide)
+    )
     (pin "1")
     (pin "2")
@@
       (effects (font (size 1.27 1.27)) hide)
     )
+    (property "LCSC Part#" "C96346" (id 4) (at 92.71 34.29 0)
+      (effects (font (size 1.27 1.27)) hide)
+    )
     (pin "1")
     (pin "2")
@@
       (effects (font (size 1.27 1.27)) hide)
     )
+    (property "LCSC Part#" "C21564" (id 4) (at 50.8 33.02 0)
+      (effects (font (size 1.27 1.27)) hide)
+    )
     (pin "1")
     (pin "2")
@@
     )
     (path "/00000000-0000-0000-0000-000061c802e4"
-      (reference "C8") (unit 1) (value "22u") (footprint "Capacitor_SMD:C_0805_2012Metric")
+      (reference "C8") (unit 1) (value "22uF") (footprint "Capacitor_SMD:C_0805_2012Metric")
     )
     (path "/00000000-0000-0000-0000-000061c8a487"
-      (reference "C9") (unit 1) (value "22u") (footprint "Capacitor_SMD:C_0805_2012Metric")
+      (reference "C9") (unit 1) (value "22uF") (footprint "Capacitor_SMD:C_0805_2012Metric")
     )
     (path "/fd3c6633-cd21-4d22-84a1-a796a98570ef"
@@
     )
     (path "/00000000-0000-0000-0000-000061da5b73"
-      (reference "R10") (unit 1) (value "4k7") (footprint "Resistor_SMD:R_0805_2012Metric")
+      (reference "R10") (unit 1) (value "4K7") (footprint "Resistor_SMD:R_0805_2012Metric")
     )
     (path "/00000000-0000-0000-0000-000061dc3c1d"
-      (reference "R11") (unit 1) (value "4k7") (footprint "Resistor_SMD:R_0805_2012Metric")
+      (reference "R11") (unit 1) (value "4K7") (footprint "Resistor_SMD:R_0805_2012Metric")
     )
     (path "/00000000-0000-0000-0000-000061dc9217"
-      (reference "R12") (unit 1) (value "4k7") (footprint "Resistor_SMD:R_0805_2012Metric")
+      (reference "R12") (unit 1) (value "4K7") (footprint "Resistor_SMD:R_0805_2012Metric")
     )
     (path "/00000000-0000-0000-0000-000061c5db06"
@@
     )
     (path "/00000000-0000-0000-0000-000061c5e1c5"
-      (reference "R16") (unit 1) (value "10k") (footprint "Resistor_SMD:R_0805_2012Metric")
+      (reference "R16") (unit 1) (value "10K") (footprint "Resistor_SMD:R_0805_2012Metric")
     )
     (path "/00000000-0000-0000-0000-000061c6b7aa"
-      (reference "R17") (unit 1) (value "10k") (footprint "Resistor_SMD:R_0805_2012Metric")
+      (reference "R17") (unit 1) (value "10K") (footprint "Resistor_SMD:R_0805_2012Metric")
     )
     (path "/00000000-0000-0000-0000-000061c6f699"
-      (reference "R18") (unit 1) (value "10k") (footprint "Resistor_SMD:R_0805_2012Metric")
+      (reference "R18") (unit 1) (value "10K") (footprint "Resistor_SMD:R_0805_2012Metric")
     )
     (path "/2af03734-769d-4be2-8727-78cbed8fec04"
-      (reference "R19") (unit 1) (value "4.7K") (footprint "Resistor_SMD:R_0805_2012Metric")
+      (reference "R19") (unit 1) (value "4K7") (footprint "Resistor_SMD:R_0805_2012Metric")
     )
     (path "/9c27bafe-dc9a-4fc8-9304-3713da742e75"
