File: kicad/orange_juice_board.kicad_sch (KiCad schematic)
At the start: 56 parts, among them J10 GPIO12_Head, J10 PWM_OUT1, J11 CONN_UART, J12 Conn_01x08, J12 PWM_OUT2, J13 GPIO6_Head, J14 GPIO11_Head, J15 PWM_OUT3, J2 DC_INPUT, J3 CONN_ADXL345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

Commit message: update to v0.7
Parts:
- L1: footprint Inductor_SMD:L_7.3x7.3_H4.5 -> Inductor_SMD:L_Abracon_ASPI-0630LR
Changed lines of the file:
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@@
     (property "Reference" "L1" (id 0) (at 208.28 26.67 90))
     (property "Value" "22uH" (id 1) (at 208.28 29.21 90))
-    (property "Footprint" "Inductor_SMD:L_7.3x7.3_H4.5" (id 2) (at 208.28 31.75 0)
+    (property "Footprint" "Inductor_SMD:L_Abracon_ASPI-0630LR" (id 2) (at 208.28 31.75 0)
       (effects (font (size 1.27 1.27)) hide)
     )
@@
     )
     (path "/68847f45-a180-4762-b13e-ddda7a221996"
-      (reference "L1") (unit 1) (value "22uH") (footprint "Inductor_SMD:L_7.3x7.3_H4.5")
+      (reference "L1") (unit 1) (value "22uH") (footprint "Inductor_SMD:L_Abracon_ASPI-0630LR")
     )
     (path "/00000000-0000-0000-0000-000061d8e441"

Commit message: update to v0.7
Parts:
- R3: value 25K -> 25K5
Changed lines of the file:
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@@
       (effects (font (size 1.27 1.27)) (justify left))
     )
-    (property "Value" "25K" (id 1) (at 90.17 45.7199 0)
+    (property "Value" "25K5" (id 1) (at 90.17 45.7199 0)
       (effects (font (size 1.27 1.27)) (justify left))
     )
@@
     )
     (path "/6d3d5a17-1dc1-4b4d-b3ac-05b8801f79eb"
-      (reference "R3") (unit 1) (value "25K") (footprint "Resistor_SMD:R_0805_2012Metric")
+      (reference "R3") (unit 1) (value "25K5") (footprint "Resistor_SMD:R_0805_2012Metric")
     )
     (path "/4a2fd7c0-d2ad-41a1-9c31-0a59644fa5ed"

Commit message: update bom
Parts:
- C1, C2: LCSC Part# (none) -> C723460
- C3: LCSC Part# (none) -> C83170
- C4: LCSC Part# (none) -> C3345
- D5: LCSC Part# (none) -> C64982
- L1: LCSC Part# (none) -> C128694
- R2: LCSC Part# (none) -> C100049
- R3: LCSC Part# (none) -> C228665
- R4: LCSC Part# (none) -> C84376
- R5: LCSC Part# (none) -> C273976
- U1, U3: LCSC Part# (none) -> C2687116
- U2: LCSC Part# (none) -> C9864
Changed lines of the file:
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@@
+      (effects (font (size 1.27 1.27)) hide)
+    )
+    (property "LCSC Part#" "C100049" (id 4) (at 87.63 36.83 0)
       (effects (font (size 1.27 1.27)) hide)
     )
@@
       (effects (font (size 1.27 1.27)) hide)
     )
+    (property "LCSC Part#" "C83170" (id 4) (at 193.04 31.75 0)
+      (effects (font (size 1.27 1.27)) hide)
+    )
     (pin "1")
     (pin "2")
@@
     )
     (property "Datasheet" "https://www.st.com/resource/en/datasheet/usblc6-2.pdf" (id 3) (at 99.06 167.64 0)
+      (effects (font (size 1.27 1.27)) hide)
+    )
+    (property "LCSC Part#" "C2687116" (id 4) (at 93.98 176.53 0)
       (effects (font (size 1.27 1.27)) hide)
     )
@@
       (effects (font (size 1.27 1.27)) hide)
     )
+    (property "LCSC Part#" "C273976" (id 4) (at 224.79 45.72 0)
+      (effects (font (size 1.27 1.27)) hide)
+    )
     (pin "1")
     (pin "2")
@@
       (effects (font (size 1.27 1.27)) hide)
     )
+    (property "LCSC Part#" "C723460" (id 4) (at 66.04 36.83 0)
+      (effects (font (size 1.27 1.27)) hide)
+    )
     (pin "1")
     (pin "2")
@@
     )
     (property "Datasheet" "https://www.st.com/resource/en/datasheet/usblc6-2.pdf" (id 3) (at 153.67 167.64 0)
+      (effects (font (size 1.27 1.27)) hide)
+    )
+    (property "LCSC Part#" "C2687116" (id 4) (at 148.59 176.53 0)
       (effects (font (size 1.27 1.27)) hide)
     )
@@
       (effects (font (size 1.27 1.27)) hide)
     )
+    (property "LCSC Part#" "C84376" (id 4) (at 224.79 38.1 0)
+      (effects (font (size 1.27 1.27)) hide)
+    )
     (pin "1")
     (pin "2")
@@
     )
     (property "Datasheet" "http://www.ti.com/lit/ds/symlink/tps5430.pdf" (id 3) (at 139.7 36.83 0)
+      (effects (font (size 1.27 1.27)) hide)
+    )
+    (property "LCSC Part#" "C9864" (id 4) (at 139.7 36.83 0)
       (effects (font (size 1.27 1.27)) hide)
     )
@@
       (effects (font (size 1.27 1.27)) hide)
     )
+    (property "LCSC Part#" "C128694" (id 4) (at 208.28 31.75 0)
+      (effects (font (size 1.27 1.27)) hide)
+    )
     (pin "1")
     (pin "2")
@@
       (effects (font (size 1.27 1.27)) hide)
     )
+    (property "LCSC Part#" "C228665" (id 4) (at 87.63 44.45 0)
+      (effects (font (size 1.27 1.27)) hide)
+    )
     (pin "1")
     (pin "2")
@@
     )
     (property "Datasheet" "~" (id 3) (at 213.36 38.1 0)
+      (effects (font (size 1.27 1.27)) hide)
+    )
+    (property "LCSC Part#" "C3345" (id 4) (at 213.36 38.1 0)
       (effects (font (size 1.27 1.27)) hide)
     )
@@
       (effects (font (size 1.27 1.27)) hide)
     )
+    (property "LCSC Part#" "C723460" (id 4) (at 76.2 36.83 0)
+      (effects (font (size 1.27 1.27)) hide)
+    )
     (pin "1")
     (pin "2")
@@
       (effects (font (size 1.27 1.27)) hide)
     )
+    (property "LCSC Part#" "C64982" (id 4) (at 201.93 38.1 0)
+      (effects (font (size 1.27 1.27)) hide)
+    )

Commit message: Reverse polarity
Connections:
- net BUCK_IN: now also J10.2 (Pin_2), J12.2 (Pin_2), J15.2 (Pin_2); no longer J10.1 (Pin_1), J12.1 (Pin_1), J15.1 (Pin_1)
- net BUCK_OUT: now also J8.2 (Pin_2), J9.2 (Pin_2); no longer J8.1 (Pin_1), J9.1 (Pin_1)
- net GND: now also J8.1 (Pin_1), J9.1 (Pin_1); no longer J8.2 (Pin_2), J9.2 (Pin_2)
- net at D2.1 (K), Q2.3 (D): now also J10.1 (Pin_1); no longer J10.2 (Pin_2)
- net at D3.1 (K), Q3.3 (D): now also J12.1 (Pin_1); no longer J12.2 (Pin_2)
- net at D4.1 (K), Q4.3 (D): now also J15.1 (Pin_1); no longer J15.2 (Pin_2)
Other:
- moved on the sheet: J10, J12, J15, J8, J9
